File: TestBoards/TestBackplane.kicad_pcb (KiCad board)
At the start: 18 copper layers, 70.6 x 95.5 mm, 12 parts, among them J1 BackplaneConn, J2 BackplaneConn, J3 BackplaneConn, J4 BackplaneConn, J5 BackplaneConn, J6 BackplaneConn, J7 BackplaneConn, J8 BackplaneConn

Commit message: Fixed via dangling, shorting vias and via snapping in KiCad export
Routing:
- net B10B11_015: track 0.00 -> 242.8 mm, vias 0 -> 5
- net B01B03_004: track 0.00 -> 214.8 mm, vias 0 -> 4
- net B00B01_013: track 0.00 -> 154.4 mm, vias 0 -> 5
- net B11B15_003: track 0.00 -> 144.8 mm, vias 0 -> 2
- net B01B05_009: track 0.00 -> 120.4 mm, vias 0 -> 2
- net B09B13_013: track 0.00 -> 119.2 mm, vias 0 -> 2
- net B12B14_002: track 0.00 -> 110.0 mm, vias 0 -> 3
- net B01B05_011: track 0.00 -> 108.4 mm, vias 0 -> 1
- net B03B07_015: track 0.00 -> 105.2 mm, vias 0 -> 4
- net B10B14_001: track 0.00 -> 100.0 mm, vias 0 -> 1
- net B08B10_005: track 0.00 -> 99.2 mm, vias 0 -> 2
- net B00B02_007: track 0.00 -> 99.2 mm, vias 0 -> 2
- net B02B06_005: track 0.00 -> 96.4 mm, vias 0 -> 1
- net B13B15_002: track 0.00 -> 96.4 mm, vias 0 -> 2
- net B09B13_002: track 0.00 -> 92.0 mm, vias 0 -> 1
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